File: salero-1.kicad_pcb (KiCad board)
At the start: 2 copper layers, 23.5 x 27.3 mm, 15 parts, among them J1 Stomp_Connector, J2 Power_Connector, Q1 2N5089

Commit message: updated to KiCad 6.0
Other:
- net class Default removed
